Commit message: Add base_footprint_link and create config file for SLAM
 * modify robot_core.xacro: add base_footprint_link
 * create mapper_params_online_async.yaml SLAM parameter file

File: sevillabot/description/robot_core.xacro (robot description, xacro)
@@ -1,4 +1,4 @@
 <?xml version="1.0"?>
-<robot xmlns:xacro="http://www.ros.org/wiki/xacro" >
+<robot xmlns:xacro="http://www.ros.org/wiki/xacro">
     <!-- MATERIALS -->
     <!-- white black light_gray dark_gray green blue red yellow orange -->
@@ -9,6 +9,14 @@
     <link name="base_link">
     </link>
+    <!-- BASE_FOOTPRINT LINK -->
+    <joint name="base_footprint_joint" type="fixed">
+        <parent link="base_link" />
+        <child link="base_footprint" />
+        <origin xyz="0 0 0" rpy="0 0 0" />
+    </joint>
+    <link name="base_footprint">
+    </link>
     <!-- CHASSIS LINK -->
-    <joint name="chassis_joint" type = "fixed">
+    <joint name="chassis_joint" type="fixed">
         <parent link="base_link" />
         <child link="chassis_link" />
@@ -18,5 +26,5 @@
         <visual>
             <geometry>
-                <box size="${box_x} ${box_y} ${box_z}"/>
+                <box size="${box_x} ${box_y} ${box_z}" />
             </geometry>
             <origin xyz="${box_x/2} 0 ${box_z/2}" />
@@ -25,5 +33,5 @@
         <collision>
             <geometry>
-                <box size="${box_x} ${box_y} ${box_z}"/>
+                <box size="${box_x} ${box_y} ${box_z}" />
             </geometry>
             <origin xyz="${box_x/2} 0 ${box_z/2}" />
@@ -37,5 +45,5 @@
     </gazebo>
     <!-- LEFT WHEEL LINK -->
-    <joint name="left_wheel_joint" type = "continuous">
+    <joint name="left_wheel_joint" type="continuous">
         <parent link="base_link" />
         <child link="left_wheel_link" />
@@ -63,5 +71,5 @@
     </gazebo>
     <!-- RIGHT WHEEL LINK -->
-    <joint name="right_wheel_joint" type = "continuous">
+    <joint name="right_wheel_joint" type="continuous">
         <parent link="base_link" />
         <child link="right_wheel_link" />
@@ -88,6 +96,6 @@
         <material>Gazebo/Blue</material>
     </gazebo>
-<!-- LEFT CASTER WHEEL LINK -->
-    <joint name="left_caster_wheel_joint" type = "fixed">
+    <!-- LEFT CASTER WHEEL LINK -->
+    <joint name="left_caster_wheel_joint" type="fixed">
         <parent link="chassis_link" />
         <child link="left_caster_wheel_link" />
@@ -115,6 +123,6 @@
         <mu2 value="0.0001" />
     </gazebo>
-<!-- RIGHT CASTER WHEEL LINK     -->
-    <joint name="right_caster_wheel_joint" type = "fixed">
+    <!-- RIGHT CASTER WHEEL LINK     -->
+    <joint name="right_caster_wheel_joint" type="fixed">
         <parent link="chassis_link" />
         <child link="right_caster_wheel_link" />
@@ -143,5 +151,5 @@
     </gazebo>
     <!-- LEFT MOTOR LINK -->
-    <joint name="left_motor_joint" type = "fixed">
+    <joint name="left_motor_joint" type="fixed">
         <parent link="base_link" />
         <child link="left_motor_link" />
@@ -176,5 +184,5 @@
     </gazebo>
     <!-- RIGHT MOTOR LINK -->
-    <joint name="right_motor_joint" type = "fixed">
+    <joint name="right_motor_joint" type="fixed">
         <parent link="base_link" />
         <child link="right_motor_link" />
