Commit message: First attempt at simulating sevillabot robot
- in robot_core.xacro:
  * add ASSY_sevillabot_base.stl mesh as visual of chassis_link
  * remove extra castor and motor links
- in properties.xacro: modify dimensions to approximately fit sevillabot, add units for clarity
- in camera.xacro: add camera_angle
- in lidar.xacro: reduce min range from 0.3 to 0.1
- Add `meshes` directory, install it in CMakeLists.txt
- in Simulation.md add notes

File: sevillabot/description/camera.xacro (robot description, xacro)
@@ -4,5 +4,5 @@
         <parent link="chassis_link"/>
         <child link="camera_link"/>
-        <origin xyz="${box_x + cam_x} 0 ${box_z + cam_z}" rpy="0.0 0.0 0.0"/>
+        <origin xyz="${box_x + cam_x} 0 ${box_z + cam_z}" rpy="0.0 ${cam_angle} 0.0"/>
     </joint>
     <link name="camera_link">

File: sevillabot/description/lidar.xacro (robot description, xacro)
@@ -38,5 +38,5 @@
                 </scan>
                 <range>
-                    <min>0.3</min>
+                    <min>0.1</min>
                     <max>12</max>
                     <resolution>0.01</resolution>

File: sevillabot/description/properties.xacro (robot description, xacro)
@@ -2,40 +2,40 @@
 <robot xmlns:xacro="http://www.ros.org/wiki/xacro" >
     <!-- box -->
-    <xacro:property name="box_x" value="0.29"/> <!-- box length -->
-    <xacro:property name="box_y" value="0.19"/> <!-- box width -->
-    <xacro:property name="box_z" value="0.124"/> <!-- box height -->
-    <xacro:property name="box_mass" value="0.05"/> <!-- box mass -->
+    <xacro:property name="box_x" value="0.26"/> <!-- box length in m -->
+    <xacro:property name="box_y" value="0.22"/> <!-- box width in m -->
+    <xacro:property name="box_z" value="0.075"/> <!-- box height in m -->
+    <xacro:property name="box_mass" value="0.05"/> <!-- box mass in Kg -->
     <!-- wheels -->
-    <xacro:property name="W_x" value="0.066"/> <!-- wheel axis x-offset from centre -->
-    <xacro:property name="W_z" value="0.022"/> <!-- wheel axis z-offset from bottom -->
-    <xacro:property name="W_y" value="0.122"/> <!-- wheel half separation -->
-    <xacro:property name="W_D" value="0.065"/> <!-- wheel diameter -->
-    <xacro:property name="W_h" value="0.026"/> <!-- wheel width -->
-    <xacro:property name="W_mass" value="0.05"/> <!-- wheel mass -->
+    <xacro:property name="W_x" value="0.0"/> <!-- wheel axis x-offset from centre in m -->
+    <xacro:property name="W_z" value="0.022"/> <!-- wheel axis z-offset from bottom in m -->
+    <xacro:property name="W_y" value="0.122"/> <!-- wheel half separation in m -->
+    <xacro:property name="W_D" value="0.065"/> <!-- wheel diameter in m -->
+    <xacro:property name="W_h" value="0.026"/> <!-- wheel width in m -->
+    <xacro:property name="W_mass" value="0.05"/> <!-- wheel mass in Kg -->
     <!-- casters -->
-    <xacro:property name="c_x" value="0.024"/> <!-- caster centre x-offset from edge -->
-    <xacro:property name="c_y" value="0.024"/> <!-- caster centre y-offset from edge -->
-    <xacro:property name="c_z" value="0.049"/> <!-- caster contact z-offset from bottom -->
-    <xacro:property name="c_D" value="0.016"/> <!-- caster diameter -->
-    <xacro:property name="c_mass" value="0.05"/> <!-- caster mass -->
+    <xacro:property name="c_x" value="0.024"/> <!-- caster centre x-offset from edge in m -->
+    <xacro:property name="c_z" value="0.04"/> <!-- caster contact z-offset from bottom in m -->
+    <xacro:property name="c_D" value="0.016"/> <!-- caster diameter in m -->
+    <xacro:property name="c_mass" value="0.05"/> <!-- caster mass in Kg -->
     <!-- motors -->
-    <xacro:property name="m_y" value="0.04"/> <!-- motor y-offset from centre-->
-    <xacro:property name="m_h" value="0.06"/> <!-- motor length -->
-    <xacro:property name="m_D" value="0.02"/> <!-- motor body diameter -->
-    <xacro:property name="m_l" value="0.009"/> <!-- motor coupling length -->
-    <xacro:property name="m_d" value="0.011"/> <!-- motor coupling diameter -->
-    <xacro:property name="m_mass" value="0.05"/> <!-- motor mass -->
+    <xacro:property name="m_y" value="0.04"/> <!-- motor y-offset from centre in m -->
+    <xacro:property name="m_h" value="0.06"/> <!-- motor length in m -->
+    <xacro:property name="m_D" value="0.02"/> <!-- motor body diameter in m -->
+    <xacro:property name="m_l" value="0.009"/> <!-- motor coupling length in m -->
+    <xacro:property name="m_d" value="0.011"/> <!-- motor coupling diameter in m -->
+    <xacro:property name="m_mass" value="0.05"/> <!-- motor mass in Kg -->
     <!--lidar -->
-    <xacro:property name="L_x" value="0.0"/> <!-- Lidar x-offset from box centre -->
-    <xacro:property name="L_z" value="0.023"/> <!-- Lidar z-offset from box top -->
-    <xacro:property name="L_D" value="0.038"/> <!-- Lidar head diameter -->
-    <xacro:property name="L_h" value="0.013"/> <!-- Lidar unit height -->
-    <xacro:property name="L_mass" value="0.0042"/> <!-- Lidar mass -->
+    <xacro:property name="L_x" value="0.16"/> <!-- Lidar x-offset from box centre in m -->
+    <xacro:property name="L_z" value="-0.055"/> <!-- Lidar z-offset from box top in m -->
+    <xacro:property name="L_D" value="0.038"/> <!-- Lidar head diameter in m -->
+    <xacro:property name="L_h" value="0.013"/> <!-- Lidar unit height in m -->
+    <xacro:property name="L_mass" value="0.0042"/> <!-- Lidar mass in Kg -->
     <!--camera -->
-    <xacro:property name="cam_x" value="0.0"/> <!-- Camera x-offset from box front face -->
-    <xacro:property name="cam_z" value="-0.03"/> <!-- Lidar z-offset from box top -->
-    <xacro:property name="cam_dx" value="0.01"/> <!-- Camera box thickness -->
-    <xacro:property name="cam_dy" value="0.04"/> <!-- Camera box width -->
-    <xacro:property name="cam_dz" value="0.03"/> <!-- Camera box height -->
-    <xacro:property name="cam_mass" value="0.002"/> <!-- Camera mass -->
+    <xacro:property name="cam_x" value="0.0"/> <!-- Camera x-offset from box front face in m -->
+    <xacro:property name="cam_z" value="-0.04"/> <!-- Camera z-offset from box top in m -->
+    <xacro:property name="cam_angle" value="${10*pi/180}"/> <!-- Camera down angle in radians -->
+    <xacro:property name="cam_dx" value="0.01"/> <!-- Camera box thickness in m -->
+    <xacro:property name="cam_dy" value="0.04"/> <!-- Camera box width in m -->
+    <xacro:property name="cam_dz" value="0.03"/> <!-- Camera box height in m -->
+    <xacro:property name="cam_mass" value="0.002"/> <!-- Camera mass in Kg -->
 </robot>

File: sevillabot/description/robot_core.xacro (robot description, xacro)
@@ -26,7 +26,8 @@
         <visual>
             <geometry>
-                <box size="${box_x} ${box_y} ${box_z}" />
+            	<mesh filename="file://$(find sevillabot)/meshes/ASSY_sevillabot_base.stl" scale="1.0e-3 1.0e-3 1.0e-3"/>
+                <!-- box size="${box_x} ${box_y} ${box_z}" /> -->
             </geometry>
-            <origin xyz="${box_x/2} 0 ${box_z/2}" />
+            <origin xyz="${box_x/2} 0 0" rpy="0 0 -${pi/2}"/>
             <material name="white" />
         </visual>
@@ -96,11 +97,11 @@
         <material>Gazebo/Blue</material>
     </gazebo>
-    <!-- LEFT CASTER WHEEL LINK -->
-    <joint name="left_caster_wheel_joint" type="fixed">
+    <!-- CASTER WHEEL LINK -->
+    <joint name="caster_wheel_joint" type="fixed">
         <parent link="chassis_link" />
-        <child link="left_caster_wheel_link" />
-        <origin xyz="${box_x-c_x} ${box_y/2-c_y} ${-c_z}" />
+        <child link="caster_wheel_link" />
+        <origin xyz="${box_x-c_x} 0 ${-c_z}" />
     </joint>
-    <link name="left_caster_wheel_link">
+    <link name="caster_wheel_link">
         <visual>
             <geometry>
@@ -118,101 +119,8 @@
         </xacro:inertial_sphere>
     </link>
-    <gazebo reference="left_caster_wheel_link">
+    <gazebo reference="caster_wheel_link">
         <material>Gazebo/Yellow</material>
         <mu1 value="0.0001" />
         <mu2 value="0.0001" />
     </gazebo>
-    <!-- RIGHT CASTER WHEEL LINK     -->
-    <joint name="right_caster_wheel_joint" type="fixed">
-        <parent link="chassis_link" />
-        <child link="right_caster_wheel_link" />
-        <origin xyz="${box_x-c_x} ${-box_y/2+c_y} ${-c_z}" />
-    </joint>
-    <link name="right_caster_wheel_link">
-        <visual>
-            <geometry>
-                <sphere radius="${c_D/2}" />
-            </geometry>
-            <material name="yellow" />
-        </visual>
-        <collision>
-            <geometry>
-                <sphere radius="${c_D/2}" />
-            </geometry>
-        </collision>
-        <xacro:inertial_sphere mass="${c_mass}" radius="${c_D/2}">
-            <origin xyz="0 0 0" rpy="0 0 0" />
-        </xacro:inertial_sphere>
-    </link>
-    <gazebo reference="right_caster_wheel_link">
-        <material>Gazebo/Yellow</material>
-        <mu1 value="0.0001" />
-        <mu2 value="0.0001" />
-    </gazebo>
-    <!-- LEFT MOTOR LINK -->
-    <joint name="left_motor_joint" type="fixed">
-        <parent link="base_link" />
-        <child link="left_motor_link" />
-        <origin xyz="0 ${m_y+m_h/2} 0" rpy="-${pi/2} 0 0" />
-    </joint>
-    <link name="left_motor_link">
-        <visual>
-            <geometry>
-                <cylinder radius="${m_D/2}" length="${m_h}" />
-            </geometry>
-            <origin xyz="0 0 0" />
-            <material name="red" />
-        </visual>
-        <visual>
-            <geometry>
-                <cylinder radius="${m_d/2}" length="${m_l}" />
-            </geometry>
-            <origin xyz="0 0 ${(m_h+m_l)/2}" />
-            <material name="red" />
-        </visual>
-        <collision>
-            <geometry>
-                <cylinder radius="${m_D/2}" length="${m_h}" />
-            </geometry>
-        </collision>
-        <xacro:inertial_cylinder mass="${m_mass}" radius="${m_D/2}" length="${m_h}">
-            <origin xyz="0 0 0" rpy="0 0 0" />
-        </xacro:inertial_cylinder>
-    </link>
-    <gazebo reference="left_motor_link">
-        <material>Gazebo/Red</material>
-    </gazebo>
-    <!-- RIGHT MOTOR LINK -->
-    <joint name="right_motor_joint" type="fixed">
-        <parent link="base_link" />
-        <child link="right_motor_link" />
-        <origin xyz="0 -${m_y+m_h/2} 0" rpy="${pi/2} 0 0" />
-    </joint>
-    <link name="right_motor_link">
-        <visual>
-            <geometry>
-                <cylinder radius="${m_D/2}" length="${m_h}" />
-            </geometry>
-            <origin xyz="0 0 0" />
-            <material name="red" />
-        </visual>
-        <visual>
-            <geometry>
-                <cylinder radius="${m_d/2}" length="${m_l}" />
-            </geometry>
-            <origin xyz="0 0 ${(m_h+m_l)/2}" />
-            <material name="red" />
-        </visual>
-        <collision>
-            <geometry>
-                <cylinder radius="${m_D/2}" length="${m_h}" />
-            </geometry>
-        </collision>
-        <xacro:inertial_cylinder mass="${m_mass}" radius="${m_D/2}" length="${m_h}">
-            <origin xyz="0 0 0" rpy="0 0 0" />
-        </xacro:inertial_cylinder>
-    </link>
-    <gazebo reference="right_motor_link">
-        <material>Gazebo/Red</material>
-    </gazebo>
 </robot>

Commit message: Improce simulation for sevillabot
- Add .stl files in meshes folder for base, wheels, camera, lidar
  Note: .stl files correspond to version sevillabot_v1.8_animated.FCStd
- Fine-tune .xacro files to properly render meshes, collisions,
 and inertias

File: sevillabot/description/camera.xacro (robot description, xacro)
@@ -4,12 +4,12 @@
         <parent link="chassis_link"/>
         <child link="camera_link"/>
-        <origin xyz="${box_x + cam_x} 0 ${box_z + cam_z}" rpy="0.0 ${cam_angle} 0.0"/>
+        <origin xyz="${cam_x} 0 ${cam_z}" rpy="0.0 ${cam_angle} 0.0"/>
     </joint>
     <link name="camera_link">
         <visual>
             <geometry>
-                <box size="${cam_dx} ${cam_dy} ${cam_dz}"/>
+                <mesh filename="file://$(find sevillabot)/meshes/ADDON_front_camera.stl" scale="1.0e-3 1.0e-3 1.0e-3"/>
             </geometry>
-            <origin xyz="${cam_dx/2} 0 ${cam_dz/2}" />
+            <origin xyz="0 0 0" rpy="0.0 0.0 0.0"/>
             <material name="orange" />
         </visual>
@@ -18,8 +18,8 @@
                 <box size="${cam_dx} ${cam_dy} ${cam_dz}"/>
             </geometry>
-            <origin xyz="${cam_dx/2} 0 ${cam_dz/2}" />
+            <origin xyz="0.0 0.0 0.0" />
         </collision>
         <xacro:inertial_box mass="${cam_mass}" x="${cam_dx}" y="${cam_dy}" z="${cam_dz}">
-            <origin xyz="${cam_dx/2} 0 ${cam_dz/2}" rpy="0 0 0" />
+            <origin xyz="0 0 0" rpy="0 0 0" />
         </xacro:inertial_box>
     </link>

File: sevillabot/description/lidar.xacro (robot description, xacro)
@@ -4,11 +4,12 @@
         <parent link="chassis_link"/>
         <child link="lidar_link"/>
-        <origin xyz="${box_x/2 + L_x} 0 ${box_z + L_z}" rpy="0.0 0.0 0.0"/>
+        <origin xyz="${L_x+L_x_off} 0 ${L_z+L_z_off}" rpy="0.0 0.0 0.0"/>
     </joint>
     <link name="lidar_link">
         <visual>
             <geometry>
-                <cylinder radius="${L_D/2}" length="${L_h}" />
+                <mesh filename="file://$(find sevillabot)/meshes/ADDON_Lidar_assy.stl" scale="1.0e-3 1.0e-3 1.0e-3"/>
             </geometry>
+            <origin xyz="${-L_x_off} 0 ${-L_z_off}" rpy="0.0 0.0 0.0"/>
             <material name="green" />
         </visual>
@@ -17,4 +18,5 @@
                 <cylinder radius="${L_D/2}" length="${L_h}" />
             </geometry>
+            <origin xyz="0 0 0" rpy="0 0 0" />
         </collision>
         <xacro:inertial_cylinder mass="${L_mass}" radius="${L_D/2}" length="${L_h}">

File: sevillabot/description/properties.xacro (robot description, xacro)
@@ -5,17 +5,21 @@
     <xacro:property name="box_y" value="0.22"/> <!-- box width in m -->
     <xacro:property name="box_z" value="0.075"/> <!-- box height in m -->
-    <xacro:property name="box_mass" value="0.05"/> <!-- box mass in Kg -->
+    <xacro:property name="box_x_off" value="0.0"/> <!-- box x-offset in m -->
+    <xacro:property name="box_z_off" value="0.0"/> <!-- box z-offset in m -->
+    <xacro:property name="box_mass" value="1.7578"/> <!-- box mass in Kg -->
     <!-- wheels -->
-    <xacro:property name="W_x" value="0.0"/> <!-- wheel axis x-offset from centre in m -->
-    <xacro:property name="W_z" value="0.022"/> <!-- wheel axis z-offset from bottom in m -->
-    <xacro:property name="W_y" value="0.122"/> <!-- wheel half separation in m -->
+    <xacro:property name="W_x" value="0.04"/> <!-- wheel axis x-offset from centre in m -->
+    <xacro:property name="W_z" value="0.025"/> <!-- wheel axis z-offset from bottom in m -->
+    <xacro:property name="W_y" value="0.102"/> <!-- wheel half separation in m -->
     <xacro:property name="W_D" value="0.065"/> <!-- wheel diameter in m -->
     <xacro:property name="W_h" value="0.026"/> <!-- wheel width in m -->
-    <xacro:property name="W_mass" value="0.05"/> <!-- wheel mass in Kg -->
-    <!-- casters -->
-    <xacro:property name="c_x" value="0.024"/> <!-- caster centre x-offset from edge in m -->
-    <xacro:property name="c_z" value="0.04"/> <!-- caster contact z-offset from bottom in m -->
+    <xacro:property name="W_mass" value="0.0454"/> <!-- wheel mass in Kg -->
+    <!-- caster -->
+    <xacro:property name="c_x" value="0.030"/> <!-- caster centre x-offset from edge in m -->
+    <xacro:property name="c_z" value="0.056"/> <!-- caster contact z-offset from bottom in m -->
+    <xacro:property name="c_x_off" value="0.090"/> <!-- caster mesh x-offset in m -->
+    <xacro:property name="c_z_off" value="0.043"/> <!-- caster mesh z-offset in m -->
     <xacro:property name="c_D" value="0.016"/> <!-- caster diameter in m -->
-    <xacro:property name="c_mass" value="0.05"/> <!-- caster mass in Kg -->
+    <xacro:property name="c_mass" value="0.0471"/> <!-- caster mass in Kg -->
     <!-- motors -->
     <xacro:property name="m_y" value="0.04"/> <!-- motor y-offset from centre in m -->
@@ -26,16 +30,18 @@
     <xacro:property name="m_mass" value="0.05"/> <!-- motor mass in Kg -->
     <!--lidar -->
-    <xacro:property name="L_x" value="0.16"/> <!-- Lidar x-offset from box centre in m -->
-    <xacro:property name="L_z" value="-0.055"/> <!-- Lidar z-offset from box top in m -->
+    <xacro:property name="L_x" value="0.109"/> <!-- Lidar x-offset in m -->
+    <xacro:property name="L_z" value="-0.004"/> <!-- Lidar z-offset in m -->
+    <xacro:property name="L_x_off" value="0.04"/> <!-- Lidar x-offset in m -->
+    <xacro:property name="L_z_off" value="0.022"/> <!-- Lidar z-offset in m -->
     <xacro:property name="L_D" value="0.038"/> <!-- Lidar head diameter in m -->
     <xacro:property name="L_h" value="0.013"/> <!-- Lidar unit height in m -->
-    <xacro:property name="L_mass" value="0.0042"/> <!-- Lidar mass in Kg -->
+    <xacro:property name="L_mass" value="0.0715"/> <!-- Lidar mass in Kg -->
     <!--camera -->
-    <xacro:property name="cam_x" value="0.0"/> <!-- Camera x-offset from box front face in m -->
-    <xacro:property name="cam_z" value="-0.04"/> <!-- Camera z-offset from box top in m -->
+    <xacro:property name="cam_x" value="0.127"/> <!-- Camera x-offset in m -->
+    <xacro:property name="cam_z" value="0.05216"/> <!-- Camera z-offset in m -->
     <xacro:property name="cam_angle" value="${10*pi/180}"/> <!-- Camera down angle in radians -->
-    <xacro:property name="cam_dx" value="0.01"/> <!-- Camera box thickness in m -->
-    <xacro:property name="cam_dy" value="0.04"/> <!-- Camera box width in m -->
-    <xacro:property name="cam_dz" value="0.03"/> <!-- Camera box height in m -->
+    <xacro:property name="cam_dx" value="0.006"/> <!-- Camera box thickness in m -->
+    <xacro:property name="cam_dy" value="0.03"/> <!-- Camera box width in m -->
+    <xacro:property name="cam_dz" value="0.02"/> <!-- Camera box height in m -->
     <xacro:property name="cam_mass" value="0.002"/> <!-- Camera mass in Kg -->
 </robot>

File: sevillabot/description/robot_core.xacro (robot description, xacro)
@@ -8,5 +8,5 @@
     <!-- BASE LINK -->
     <link name="base_link">
-    </link>
+    </link>length
     <!-- BASE_FOOTPRINT LINK -->
     <joint name="base_footprint_joint" type="fixed">
@@ -21,5 +21,5 @@
         <parent link="base_link" />
         <child link="chassis_link" />
-        <origin xyz="${W_x-box_x/2} 0 ${W_z}" />
+        <origin xyz="0 0 0" />
     </joint>
     <link name="chassis_link">
@@ -27,7 +27,6 @@
             <geometry>
             	<mesh filename="file://$(find sevillabot)/meshes/ASSY_sevillabot_base.stl" scale="1.0e-3 1.0e-3 1.0e-3"/>
-                <!-- box size="${box_x} ${box_y} ${box_z}" /> -->
             </geometry>
-            <origin xyz="${box_x/2} 0 0" rpy="0 0 -${pi/2}"/>
+            <origin xyz="${box_z_off} 0 ${box_z_off}" rpy="0 0 0"/>
             <material name="white" />
         </visual>
@@ -36,8 +35,8 @@
                 <box size="${box_x} ${box_y} ${box_z}" />
             </geometry>
-            <origin xyz="${box_x/2} 0 ${box_z/2}" />
+            <origin xyz="0 0 ${box_z/2}" />
         </collision>
         <xacro:inertial_box mass="${box_mass}" x="${box_x}" y="${box_y}" z="${box_z}">
-            <origin xyz="${box_x/2} 0 ${box_z/2}" rpy="0 0 0" />
+            <origin xyz="0 0 0" rpy="0 0 0" />
         </xacro:inertial_box>
     </link>
@@ -49,11 +48,11 @@
         <parent link="base_link" />
         <child link="left_wheel_link" />
-        <origin xyz="0 ${W_y} 0" rpy="-${pi/2} 0 0" />
-        <axis xyz="0 0 1" />
+        <origin xyz="-${W_x} ${W_y} -${W_z}" rpy="0 0 ${pi/2}" />
+        <axis xyz="1 0 0" />
     </joint>
     <link name="left_wheel_link">
         <visual>
             <geometry>
-                <cylinder radius="${W_D/2}" length="${W_h}" />
+                <mesh filename="file://$(find sevillabot)/meshes/ASSY_Wheel.stl" scale="1.0e-3 1.0e-3 1.0e-3"/>
             </geometry>
             <material name="blue" />
@@ -65,5 +64,5 @@
         </collision>
         <xacro:inertial_cylinder mass="${W_mass}" radius="${W_D/2}" length="${W_h}">
-            <origin xyz="0 0 0" rpy="0 0 0" />
+            <origin xyz="0 0 0" rpy="${pi/2} 0 ${pi/2}" />
         </xacro:inertial_cylinder>
     </link>
@@ -75,11 +74,12 @@
         <parent link="base_link" />
         <child link="right_wheel_link" />
-        <origin xyz="0 -${W_y} 0" rpy="${pi/2} 0 0" />
-        <axis xyz="0 0 -1" />
+        <origin xyz="-${W_x} -${W_y} -${W_z}" rpy="0 0 -${pi/2}" />
+        <axis xyz="-1 0 0" />
     </joint>
     <link name="right_wheel_link">
         <visual>
             <geometry>
-                <cylinder radius="${W_D/2}" length="${W_h}" />
+                <!-- cylinder radius="${W_D/2}" length="${W_h}" / -->
+                <mesh filename="file://$(find sevillabot)/meshes/ASSY_Wheel.stl" scale="1.0e-3 1.0e-3 1.0e-3"/>
             </geometry>
             <material name="blue" />
@@ -91,5 +91,5 @@
         </collision>
         <xacro:inertial_cylinder mass="${W_mass}" radius="${W_D/2}" length="${W_h}">
-            <origin xyz="0 0 0" rpy="0 0 0" />
+            <origin xyz="0 0 0" rpy="${pi/2} 0 ${pi/2}" />
         </xacro:inertial_cylinder>
     </link>
@@ -101,14 +101,17 @@
         <parent link="chassis_link" />
         <child link="caster_wheel_link" />
-        <origin xyz="${box_x-c_x} 0 ${-c_z}" />
+        <origin xyz="${c_x_off} 0 ${-c_z_off}" rpy = "0 0 0"  />
     </joint>
     <link name="caster_wheel_link">
         <visual>
             <geometry>
-                <sphere radius="${c_D/2}" />
+                <!-- sphere radius="${c_D/2}" / -->
+                <mesh filename="file://$(find sevillabot)/meshes/ADDON_caster_wheel.stl" scale="1.0e-3 1.0e-3 1.0e-3"/>
             </geometry>
+            <origin xyz="0 0 0" rpy = "0 0 0"  />
             <material name="yellow" />
         </visual>
         <collision>
+            <origin xyz="0 0 0" rpy="0 0 0" />
             <geometry>
                 <sphere radius="${c_D/2}" />
