Commit message: Fine tune Simulation
* In `properties.xacro` fix bug: `W_z` (wheel axis z-offset in m) = 0.02
  (not 0.025, otherwise wheels are out of their axes!)
  Confirmed that this matches FreeCAD reference frame displacement.
* Modify `launch_sim.launch.py`to load `sevillabot_world.world` as default
  world for gazebo simulation
* Add default RVIZ config `display_bot.rviz`
* In `camera.xacro`:
   - modify horizontal FOV to 160 degrees.
   - since camera is small, remove <collision> and <inertial> tags.
* Update `Camera.md` with camera properties
* In `Simulation.md` add notes for teleop with joystick and all changes above

File: sevillabot/description/camera.xacro (robot description, xacro)
@@ -14,13 +14,4 @@
             <material name="orange" />
         </visual>
-        <collision>
-            <geometry>
-                <box size="${cam_dx} ${cam_dy} ${cam_dz}"/>
-            </geometry>
-            <origin xyz="0.0 0.0 0.0" />
-        </collision>
-        <xacro:inertial_box mass="${cam_mass}" x="${cam_dx}" y="${cam_dy}" z="${cam_dz}">
-            <origin xyz="0 0 0" rpy="0 0 0" />
-        </xacro:inertial_box>
     </link>
     <joint name="camera_optical_joint" type="fixed">
@@ -37,5 +28,5 @@
             <update_rate>10</update_rate>
             <camera>
-                <horizontal_fov>1.086</horizontal_fov> <!-- 62.2deg PiCamera-->
+                <horizontal_fov>5.671</horizontal_fov> <!-- Sensor Omnivision 5647 angle 160deg -->
                 <image>
                     <format>R8G8B8</format>

File: sevillabot/description/properties.xacro (robot description, xacro)
@@ -10,5 +10,5 @@
     <!-- wheels -->
     <xacro:property name="W_x" value="0.04"/> <!-- wheel axis x-offset from centre in m -->
-    <xacro:property name="W_z" value="0.025"/> <!-- wheel axis z-offset from bottom in m -->
+    <xacro:property name="W_z" value="0.02"/> <!-- wheel axis z-offset from bottom in m -->
     <xacro:property name="W_y" value="0.102"/> <!-- wheel half separation in m -->
     <xacro:property name="W_D" value="0.065"/> <!-- wheel diameter in m -->
